File: Interface Design/DE0/CoCo_FPGA_Hat.kicad_sch (KiCad schematic)
At the start: 16 parts, among them J1 J1, P1 CoCo_Slot, U1 74LVC245A, U2 74LVC245A, U3 74LVC245A, U4 74LVC245A

Commit message: REvised PCB for CoCo, added DE0 version
Parts:
- IDC1: value DE1 GPIO -> DE0 GPIO
- P1: footprint Roni Footprints:COCO-CART-HAT -> CoCoEPROMpak:COCO-CART-2.1X1.75; symbol Roni Symbols:CoCo_Slot -> Roni Symbols:CoCo_Slot_BarePCB
Connections:
- net *C_CTS: now also IDC1.7 (Pin_7); no longer IDC1.5 (Pin_5)
- net C_A0: now also IDC1.20 (Pin_20); no longer IDC1.21 (Pin_21)
- net C_A10: now also IDC1.15 (Pin_15); no longer IDC1.17 (Pin_17)
- net C_A12: now also IDC1.14 (Pin_14); no longer IDC1.18 (Pin_18)
- net C_A14: now also IDC1.5 (Pin_5); no longer IDC1.1 (Pin_1)
- net C_A3: now also IDC1.13 (Pin_13); no longer IDC1.9 (Pin_9)
- net C_A6: now also IDC1.18 (Pin_18); no longer IDC1.19 (Pin_19)
- net C_A8: now also IDC1.16 (Pin_16); no longer IDC1.20 (Pin_20)
- net C_A9: now also IDC1.9 (Pin_9); no longer IDC1.7 (Pin_7)
- net /C_BUSDIR: now also IDC1.17 (Pin_17); no longer IDC1.15 (Pin_15)
- net +5V: no longer names the net of P1.9 (+5V)
- no-connect marks 5 -> 9
Other:
- title: CoCo DE1 Hat -> CoCo FPGA Hat (DE0 Version)
Changed lines of the file:
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@@
   (paper "A4" portrait)
   (title_block
-    (title "CoCo DE1 Hat")
-    (date "2023-01-15")
+    (title "CoCo FPGA Hat (DE0 Version)")
+    (date "2023-01-16")
     (rev "Rev 0")
     (company "RCC")
     (comment 1 "to 3.3v systems with voltage conversion")
     (comment 2 "Cartridge for TRS-80 Color Computers that expose the Computer BUS")
-    (comment 3 "IDC connector pinout mapped for Altera DE1 FPGA Development Board")
+    (comment 3 "IDC connector pinout mapped for Altera DE0 FPGA Development Board")
   )
   (junction (at 167.386 106.172) (diameter 0) (color 0 0 0 0)
@@
   (junction (at 117.7027 166.751) (diameter 0) (color 0 0 0 0)
   )
+  (no_connect (at 154.178 47.498))
   (no_connect (at 60.96 112.776))
+  (no_connect (at 154.178 72.898))
   (no_connect (at 45.72 41.656))
+  (no_connect (at 40.64 41.656))
   (no_connect (at 154.178 60.198))
+  (no_connect (at 154.178 70.358))
   (no_connect (at 30.48 107.696))
   (no_connect (at 50.8 41.656))
@@
     )
   )
-  (global_label "{slash}C_BUSDIR" (shape input) (at 154.178 65.278 180) (fields_autoplaced)
-    (effects (font (size 1 1)) (justify right))
-    (property "Intersheet References" "${INTERSHEET_REFS}" (id 0) (at 141.242 65.1986 0)
+  (global_label "{slash}C_BUSDIR" (shape input) (at 154.178 67.818 180) (fields_autoplaced)
+    (effects (font (size 1 1)) (justify right))
+    (property "Intersheet References" "${INTERSHEET_REFS}" (id 0) (at 141.242 67.7386 0)
       (effects (font (size 1 1)) (justify right) hide)
     )
@@
     )
   )
-  (global_label "C_A0" (shape input) (at 154.178 72.898 180) (fields_autoplaced)
-    (effects (font (size 1 1)) (justify right))
-    (property "Intersheet References" "${INTERSHEET_REFS}" (id 0) (at 150.348 72.9417 0)
-      (effects (font (size 1 1)) (justify right) hide)
+  (global_label "C_A0" (shape input) (at 166.878 70.358 0) (fields_autoplaced)
+    (effects (font (size 1 1)) (justify left))
+    (property "Intersheet References" "${INTERSHEET_REFS}" (id 0) (at 170.708 70.3143 0)
+      (effects (font (size 1 1)) (justify left) hide)
     )
   )
@@
     )
   )
-  (global_label "C_A10" (shape input) (at 154.178 67.818 180) (fields_autoplaced)
-    (effects (font (size 1 1)) (justify right))
-    (property "Intersheet References" "${INTERSHEET_REFS}" (id 0) (at 149.6813 67.8617 0)
-      (effects (font (size 1 1)) (justify right) hide)
-    )
-  )
-  (global_label "C_A9" (shape input) (at 154.178 55.118 180) (fields_autoplaced)
-    (effects (font (size 1 1)) (justify right))
-    (property "Intersheet References" "${INTERSHEET_REFS}" (id 0) (at 150.348 55.1617 0)
+  (global_label "C_A10" (shape input) (at 154.178 65.278 180) (fields_autoplaced)
+    (effects (font (size 1 1)) (justify right))
+    (property "Intersheet References" "${INTERSHEET_REFS}" (id 0) (at 149.6813 65.3217 0)
+      (effects (font (size 1 1)) (justify right) hide)
+    )
+  )
+  (global_label "C_A9" (shape input) (at 154.178 57.658 180) (fields_autoplaced)
+    (effects (font (size 1 1)) (justify right))
+    (property "Intersheet References" "${INTERSHEET_REFS}" (id 0) (at 150.348 57.7017 0)
       (effects (font (size 1 1)) (justify right) hide)
     )
@@
     )
   )
-  (global_label "*C_CTS" (shape input) (at 154.178 52.578 180) (fields_autoplaced)
-    (effects (font (size 1 1)) (justify right))
-    (property "Intersheet References" "${INTERSHEET_REFS}" (id 0) (at 147.0399 52.6405 0)
+  (global_label "*C_CTS" (shape input) (at 154.178 55.118 180) (fields_autoplaced)
+    (effects (font (size 1 1)) (justify right))
+    (property "Intersheet References" "${INTERSHEET_REFS}" (id 0) (at 147.0399 55.1805 0)
       (effects (font (size 1 1)) (justify right) hide)
     )
@@
     )
   )
-  (global_label "C_A8" (shape input) (at 166.878 70.358 0) (fields_autoplaced)
-    (effects (font (size 1 1)) (justify left))
-    (property "Intersheet References" "${INTERSHEET_REFS}" (id 0) (at 170.708 70.3143 0)
+  (global_label "C_A8" (shape input) (at 166.878 65.278 0) (fields_autoplaced)
+    (effects (font (size 1 1)) (justify left))
+    (property "Intersheet References" "${INTERSHEET_REFS}" (id 0) (at 170.708 65.2343 0)
       (effects (font (size 1 1)) (justify left) hide)
     )
@@
     )
   )
-  (global_label "C_A3" (shape input) (at 154.178 57.658 180) (fields_autoplaced)
-    (effects (font (size 1 1)) (justify right))
-    (property "Intersheet References" "${INTERSHEET_REFS}" (id 0) (at 150.348 57.7017 0)
+  (global_label "C_A3" (shape input) (at 154.178 62.738 180) (fields_autoplaced)
+    (effects (font (size 1 1)) (justify right))
+    (property "Intersheet References" "${INTERSHEET_REFS}" (id 0) (at 150.348 62.7817 0)
       (effects (font (size 1 1)) (justify right) hide)
     )
@@
     )
   )
-  (global_label "C_A6" (shape input) (at 154.178 70.358 180) (fields_autoplaced)
-    (effects (font (size 1 1)) (justify right))
-    (property "Intersheet References" "${INTERSHEET_REFS}" (id 0) (at 150.348 70.4017 0)
-      (effects (font (size 1 1)) (justify right) hide)
-    )
-  )
-  (global_label "C_A12" (shape input) (at 166.878 67.818 0) (fields_autoplaced)
-    (effects (font (size 1 1)) (justify left))
-    (property "Intersheet References" "${INTERSHEET_REFS}" (id 0) (at 171.3747 67.7743 0)
+  (global_label "C_A6" (shape input) (at 166.878 67.818 0) (fields_autoplaced)
+    (effects (font (size 1 1)) (justify left))
+    (property "Intersheet References" "${INTERSHEET_REFS}" (id 0) (at 170.708 67.7743 0)
+      (effects (font (size 1 1)) (justify left) hide)
+    )
+  )
+  (global_label "C_A12" (shape input) (at 166.878 62.738 0) (fields_autoplaced)
+    (effects (font (size 1 1)) (justify left))
+    (property "Intersheet References" "${INTERSHEET_REFS}" (id 0) (at 171.3747 62.6943 0)
       (effects (font (size 1 1)) (justify left) hide)
     )
@@
     )
   )
-  (global_label "C_A14" (shape input) (at 154.178 47.498 180) (fields_autoplaced)
-    (effects (font (size 1 1)) (justify right))
-    (property "Intersheet References" "${INTERSHEET_REFS}" (id 0) (at 149.6813 47.5417 0)
+  (global_label "C_A14" (shape input) (at 154.178 52.578 180) (fields_autoplaced)
+    (effects (font (size 1 1)) (justify right))
+    (property "Intersheet References" "${INTERSHEET_REFS}" (id 0) (at 149.6813 52.6217 0)
       (effects (font (size 1 1)) (justify right) hide)
     )
@@
     (property "Datasheet" "" (id 3) (at 107.315 115.697 0)
       (effects (font (size 1 1)) hide)
-    )
-    (pin "1")
-  )
-  (symbol (lib_id "power:+5V") (at 40.64 41.656 0) (unit 1)
-    (in_bom yes) (on_board yes)
-    (property "Reference" "#PWR01" (id 0) (at 40.64 45.466 0)
-      (effects (font (size 1.27 1.27)) hide)
-    )
-    (property "Value" "+5V" (id 1) (at 40.386 38.1 0))
-    (property "Footprint" "" (id 2) (at 40.64 41.656 0)
-      (effects (font (size 1.27 1.27)) hide)
-    )
-    (property "Datasheet" "" (id 3) (at 40.64 41.656 0)
-      (effects (font (size 1.27 1.27)) hide)
     )
     (pin "1")
@@
     (pin "1")
   )
-  (symbol (lib_id "Roni Symbols:CoCo_Slot") (at 45.72 87.376 0) (unit 1)
+  (symbol (lib_id "Roni Symbols:CoCo_Slot_BarePCB") (at 45.72 87.376 0) (unit 1)
     (in_bom yes) (on_board yes) (fields_autoplaced)
     (property "Reference" "P1" (id 0) (at 52.8194 44.196 0)
@@
       (effects (font (size 1.27 1.27)) hide)
     )
-    (property "Footprint" "Roni Footprints:COCO-CART-HAT" (id 2) (at 45.72 87.376 0)
+    (property "Footprint" "CoCoEPROMpak:COCO-CART-2.1X1.75" (id 2) (at 45.72 87.376 0)
       (effects (font (size 1.27 1.27)) hide)
     )
@@
     (pin "8")
     (pin "9")
-    (pin "MTG1")
-    (pin "MTG2")
   )
   (symbol (lib_id "Device:R_Small_US") (at 93.472 123.698 0) (unit 1)
@@
   (symbol (lib_id "Connector_Generic:Conn_02x20_Odd_Even") (at 159.258 70.358 0) (unit 1)
     (in_bom yes) (on_board yes) (fields_autoplaced)
-    (property "Reference" "IDC1" (id 0) (at 160.528 40.894 0))
-    (property "Value" "DE1 GPIO" (id 1) (at 160.528 43.434 0))
+    (property "Reference" "IDC1" (id 0) (at 160.528 40.64 0))
+    (property "Value" "DE0 GPIO" (id 1) (at 160.528 43.18 0))
     (property "Footprint" "Connector_PinHeader_2.54mm:PinHeader_2x20_P2.54mm_Vertical" (id 2) (at 159.258 70.358 0)
       (effects (font (size 1 1)) hide)
@@
   )
   (symbol_instances
-    (path "/21ce861c-79ec-42b5-979a-4bd7c7632f41"
-      (reference "#PWR01") (unit 1) (value "+5V") (footprint "")
-    )
     (path "/e99d114a-e2a9-4210-99d7-57cc682175a0"
       (reference "#PWR05") (unit 1) (value "GNDREF") (footprint "")
@@
     )
     (path "/6f9656b3-3bfe-4b00-abcb-824b6a0202a0"
-      (reference "IDC1") (unit 1) (value "DE1 GPIO") (footprint "Connector_PinHeader_2.54mm:PinHeader_2x20_P2.54mm_Vertical")
+      (reference "IDC1") (unit 1) (value "DE0 GPIO") (footprint "Connector_PinHeader_2.54mm:PinHeader_2x20_P2.54mm_Vertical")
     )
     (path "/4b627ac7-f426-4ad6-aa9a-a3c2759a25ab"
@@
     )
     (path "/552ad639-2842-4abd-bb2c-fd942f893612"
-      (reference "P1") (unit 1) (value "CoCo_Slot") (footprint "Roni Footprints:COCO-CART-HAT")
+      (reference "P1") (unit 1) (value "CoCo_Slot") (footprint "CoCoEPROMpak:COCO-CART-2.1X1.75")
     )
     (path "/75b8a547-7dbb-4ae6-a265-87342b091832"
