File: Interface Design/DE1/CoCo_FPGA_Hat.kicad_pcb (KiCad board)
At the start: 2 copper layers, 53.3 x 44.5 mm, 18 parts, among them J1 J1, P1 CoCo_Slot, U1 74LVC245A, U2 74LVC245A, U3 74LVC245A, U4 74LVC245A

Commit message: Added gerber files
Routing:
- added copper zone on B.Cu, net GNDREF
Changed lines of the file:
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@@
   (segment (start 74.56 47.765) (end 75.695 48.9) (width 0.25) (layer "B.Cu") (net 78))
   (segment (start 74.56 40.81) (end 74.56 47.765) (width 0.25) (layer "B.Cu") (net 78))
+  (zone (net 69) (net_name "GNDREF") (layer "B.Cu") (hatch edge 0.508)
+    (connect_pads (clearance 0.508))
+    (min_thickness 0.254) (filled_areas_thickness no)
+    (fill yes (thermal_gap 0.508) (thermal_bridge_width 0.508))
+    (polygon
+      (pts
+        (xy 114.38 32.68)
+        (xy 114.38 66.79)
+        (xy 61.25 66.69)
+        (xy 61.21 32.67)
+        (xy 61.22 32.67)
+      )
+    )
+  )
 )
