File: Interface Design/DE1/CoCo_FPGA_Hat.kicad_sch (KiCad schematic)
At the start: 16 parts, among them J1 J1, P1 CoCo_Slot, U1 74LVC245A, U2 74LVC245A, U3 74LVC245A, U4 74LVC245A

Commit message: Added Gerber files
Parts:
- P1: footprint Roni Footprints:COCO-CART-HAT -> CoCoEPROMpak:COCO-CART-2.1X1.75; symbol Roni Symbols:CoCo_Slot -> Roni Symbols:CoCo_Slot_BarePCB
Changed lines of the file:
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@@
     (pin "1")
   )
-  (symbol (lib_id "Roni Symbols:CoCo_Slot") (at 45.72 87.376 0) (unit 1)
+  (symbol (lib_id "Roni Symbols:CoCo_Slot_BarePCB") (at 45.72 87.376 0) (unit 1)
     (in_bom yes) (on_board yes) (fields_autoplaced)
     (property "Reference" "P1" (id 0) (at 52.8194 44.196 0)
@@
       (effects (font (size 1.27 1.27)) hide)
     )
-    (property "Footprint" "Roni Footprints:COCO-CART-HAT" (id 2) (at 45.72 87.376 0)
+    (property "Footprint" "CoCoEPROMpak:COCO-CART-2.1X1.75" (id 2) (at 45.72 87.376 0)
       (effects (font (size 1.27 1.27)) hide)
     )
@@
     (pin "8")
     (pin "9")
-    (pin "MTG1")
-    (pin "MTG2")
   )
   (symbol (lib_id "Device:R_Small_US") (at 93.472 123.698 0) (unit 1)
@@
     )
     (path "/552ad639-2842-4abd-bb2c-fd942f893612"
-      (reference "P1") (unit 1) (value "CoCo_Slot") (footprint "Roni Footprints:COCO-CART-HAT")
+      (reference "P1") (unit 1) (value "CoCo_Slot") (footprint "CoCoEPROMpak:COCO-CART-2.1X1.75")
     )
     (path "/75b8a547-7dbb-4ae6-a265-87342b091832"
