File: Interface Design/CoCo_FPGA_Hat.kicad_pcb (KiCad board)
At the start: 2 copper layers, 53.3 x 44.5 mm, 18 parts, among them J1 J1, P1 CoCo_Slot, U1 74LVC245A, U2 74LVC245A, U3 74LVC245A, U4 74LVC245A

Commit message: Deleted DE1 design files -> DE0 is compatible with DE1 as well
Other:
- board text added: "CoCo FPGA Hat DE0/DE1 Rev.0"
- board text removed: "CoCo FPGA Hat DE0 Rev.0"
Changed lines of the file:
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@@
     (effects (font (size 0.5 0.5) (thickness 0.125)))
   )
-  (gr_text "CoCo FPGA Hat \nDE0 Rev.0" (at 114.14 65.29) (layer "F.SilkS")
+  (gr_text "CoCo FPGA Hat \nDE0/DE1 Rev.0" (at 114.14 65.29) (layer "F.SilkS")
     (effects (font (size 0.7 0.7) (thickness 0.15)) (justify right))
   )
