File: Interface Design/CoCo_FPGA_Hat.kicad_sch (KiCad schematic)
At the start: 16 parts, among them J1 J1, P1 CoCo_Slot, U1 74LVC245A, U2 74LVC245A, U3 74LVC245A, U4 74LVC245A

Commit message: Deleted DE1 design files -> DE0 is compatible with DE1 as well
Other:
- title: CoCo FPGA Hat (DE0 Version) -> CoCo FPGA Hat (DE0 & DE1 Compatible)
Changed lines of the file:
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@@
   (paper "A4" portrait)
   (title_block
-    (title "CoCo FPGA Hat (DE0 Version)")
-    (date "2023-01-16")
+    (title "CoCo FPGA Hat (DE0 & DE1 Compatible)")
+    (date "2023-01-17")
     (rev "Rev 0")
     (company "RCC")
     (comment 1 "to 3.3v systems with voltage conversion")
     (comment 2 "Cartridge for TRS-80 Color Computers that expose the Computer BUS")
-    (comment 3 "IDC connector pinout mapped for Altera DE0 FPGA Development Board")
+    (comment 3 "IDC connector pinout mapped for Altera DE0 & DE1 FPGA Development Board")
   )
   (junction (at 167.386 106.172) (diameter 0) (color 0 0 0 0)

Commit message: Some updates to revision number and silkscreen
Parts:
- IDC1: value DE0 GPIO -> DE0/DE1 GPIO
Changed lines of the file:
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@@
   (title_block
     (title "CoCo FPGA Hat (DE0 & DE1 Compatible)")
-    (date "2023-01-17")
-    (rev "Rev 0")
+    (date "2023-01-18")
+    (rev "0")
     (company "RCC")
     (comment 1 "to 3.3v systems with voltage conversion")
@@
     (in_bom yes) (on_board yes) (fields_autoplaced)
     (property "Reference" "IDC1" (id 0) (at 160.528 40.64 0))
-    (property "Value" "DE0 GPIO" (id 1) (at 160.528 43.18 0))
+    (property "Value" "DE0/DE1 GPIO" (id 1) (at 160.528 43.18 0))
     (property "Footprint" "Connector_PinHeader_2.54mm:PinHeader_2x20_P2.54mm_Vertical" (id 2) (at 159.258 70.358 0)
       (effects (font (size 1 1)) hide)
@@
     )
     (path "/6f9656b3-3bfe-4b00-abcb-824b6a0202a0"
-      (reference "IDC1") (unit 1) (value "DE0 GPIO") (footprint "Connector_PinHeader_2.54mm:PinHeader_2x20_P2.54mm_Vertical")
+      (reference "IDC1") (unit 1) (value "DE0/DE1 GPIO") (footprint "Connector_PinHeader_2.54mm:PinHeader_2x20_P2.54mm_Vertical")
     )
     (path "/4b627ac7-f426-4ad6-aa9a-a3c2759a25ab"
