File: Hardware Interface/CoCo_FPGA_Hat.kicad_sch (KiCad schematic)
At the start: 16 parts, among them J1 J1, P1 CoCo_Slot, U1 74LVC245A, U2 74LVC245A, U3 74LVC245A, U4 74LVC245A

Commit message: Renamed signal name for U1 /OE
Connections:
- net /C_BUSDIR renamed C_U1_D_OE
Changed lines of the file:
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@@
     )
   )
-  (global_label "{slash}C_BUSDIR" (shape input) (at 154.178 67.818 180) (fields_autoplaced)
-    (effects (font (size 1 1)) (justify right))
-    (property "Intersheet References" "${INTERSHEET_REFS}" (id 0) (at 141.242 67.7386 0)
+  (global_label "C_U1_D_OE" (shape input) (at 154.178 67.818 180) (fields_autoplaced)
+    (effects (font (size 1 1)) (justify right))
+    (property "Intersheet References" "${INTERSHEET_REFS}" (id 0) (at 144.0399 67.7555 0)
       (effects (font (size 1 1)) (justify right) hide)
     )
@@
     )
   )
-  (global_label "{slash}C_BUSDIR" (shape input) (at 119.5564 166.751 0) (fields_autoplaced)
-    (effects (font (size 1 1)) (justify left))
-    (property "Intersheet References" "${INTERSHEET_REFS}" (id 0) (at 132.4924 166.8304 0)
-      (effects (font (size 1 1)) (justify left) hide)
-    )
+  (global_label "C_U1_D_OE" (shape input) (at 119.5564 166.751 0) (fields_autoplaced)
+    (effects (font (size 1 1)) (justify left))
+    (property "Intersheet References" "${INTERSHEET_REFS}" (id 0) (at 129.6945 166.6885 0)
+      (effects (font (size 1 1)) (justify left) hide)
+    )
